File: MCP39F521_Breakout.kicad_pcb (KiCad board)
At the start: 2 copper layers, 35.6 x 27.9 mm, 39 parts, among them J11 Conn_01x10, J2 Conn_01x01, J4 Conn_01x01, J5 Conn_01x01, U1 MCP39F521, U2 MCP9700AT-ETT, Y1 Crystal

Commit message: Update to v7 and add elecrow BOM
Connections:
- net ~RESET renamed ~{RESET}
Other:
- board text added: "~{RESET}"
- board text removed: "~RESET"
